File: hardware/Transceiver_Power.kicad_sch (KiCad schematic)
At the start: 31 parts, among them U3 AD9361

Commit message: delete RF transceiver
Parts:
- removed C1, C12, C6, C9: 18pF, Capacitor_SMD:C_0201_0603Metric, symbol Device:C
- removed C100, C109, C110, C111, C98, C99: 0.1uF, Capacitor_SMD:C_0201_0603Metric, symbol Device:C_Small
- removed C104, C105, C112, C113, C114, C82: NFM15PC146R0G3D, Capacitor_SMD_Local:C_0402_1005Metric, symbol Device:C_Feedthrough
- removed C132, C133, C134, C136, C137: 0.1uF, Capacitor_SMD:C_0201_0603Metric, symbol Device:C
- removed FB2, FB3, FB4, FB5, FB6, FB7, FB8: FerriteBead_Small, Capacitor_SMD:C_0201_0603Metric, symbol Device:FerriteBead_Small
- removed R11, R12: 14.3K, Resistor_SMD:R_0201_0603Metric, symbol Device:R
- removed U3: AD9361, RF_Transceiver:bga-100_10_10_1p32_0p8, symbol 7z010_ddr:AD9361
Other:
- note removed: "1.8V"
